File: PCB Files/TinyTetris.kicad_sch (KiCad schematic)
At the start: 11 parts, among them SW1 SW_Push, SW2 SW_Push, SW3 SW_Push, SW5 SW_SPDT, U1 ATTINY85-20PU

Commit message: Update PCB Files
The PCB is thinner, the power LED was removed, and the power switch is a different type
Parts:
- removed D1: LED, LED_SMD:LED_1206_3216Metric, symbol Device:LED
- removed R6: 470, Resistor_SMD:R_0402_1005Metric, symbol Device:R
- removed SW5: SW_SPDT, Connector_PinHeader_2.54mm:PinHeader_1x03_P2.54mm_Vertical, symbol Switch:SW_SPDT
- added SW4: PCM12SMTR, footprints:SW_PCM12SMTR, symbol PCM12SMTR:PCM12SMTR
Connections:
- net GND: now also SW4.3, SW4.S1 (SHIELD), SW4.S2 (SHIELD), SW4.S3 (SHIELD), SW4.S4 (SHIELD)
- net VBUS: now also SW4.1
- net VCC: now also SW4.2
